File: MdkController.brd (EAGLE design)
At the start: 98.7 x 53.3 mm, 25 parts, among them M1 SILENTSTEPSTICK, M2 SILENTSTEPSTICK, M3 SILENTSTEPSTICK, M4 SILENTSTEPSTICK, M5 NRF8001-BREAKOUT, U1 ACPL-227, X1 1501_04, X2 1501_04, X3 1501_04

Commit message: Überarbeitung (4. Stepper entfernt, etwas aufgeräumt)
Parts:
- removed JP4: (no value), pinhead:1X04
- removed M4: SILENTSTEPSTICK, watterott:SILENTSTEPSTICK
- removed SJ1: (no value), jumper:SJ
- moved D1 1.27 mm to (22.9, 5.33)
- moved D2 1.27 mm to (19.3, 5.33)
- moved M5 1.27 mm to (40.6, 22.9)
- moved LSP1 1.09 mm to (13.1, 7.24)
- moved D4 0.64 mm to (19.6, 13.8)
- moved D5 0.64 mm to (23.1, 13.8)
- moved D6 0.64 mm to (26.7, 13.8)
- moved M2 0.64 mm to (71.1, 18.4)
- moved D3 0.63 mm to (16.0, 13.8)
- moved M1 0.63 mm to (88.9, 34.9)
- moved M3 0.63 mm to (66.0, 34.9)
Connections:
- removed net N$20: JP4.1, M4.11
- removed net N$21: JP4.2, M4.12
- removed net N$22: JP4.3, M4.13
- removed net N$23: JP4.4, M4.14
- removed net N$6: M2.9
- removed net SM4_CFG1: M4.2, U$1.45
- removed net SM4_CFG2: M4.3, U$1.46
- removed net SM4_DIR: M4.8, U$1.47
- removed net SM4_EN: M4.1, U$1.44
- removed net SM4_STEP: M4.7, U$1.5
- net 3V3: no longer M4.10
- net GND: now also M2.9; no longer M4.15, M4.9
- net VIN: no longer SJ1.2
- net VMOT: no longer M4.16, SJ1.1
Routing:
- net SM4_STEP: track 65.2 -> 0.00 mm, vias 3 -> 0
- net SM4_EN: track 51.5 -> 0.00 mm
- net SM4_CFG1: track 51.5 -> 0.00 mm
- net SM4_CFG2: track 45.4 -> 0.00 mm
- net SM4_DIR: track 35.2 -> 0.00 mm
- net VIN: track 16.3 -> 0.00 mm, vias 1 -> 0
- net N$23: track 4.97 -> 0.00 mm
- net N$22: track 4.97 -> 0.00 mm
- net N$21: track 4.97 -> 0.00 mm
- net N$20: track 4.97 -> 0.00 mm
- net 3V3: track 130.5 -> 127.7 mm
- net SM2_STEP: track 90.5 -> 92.8 mm, vias 3 -> 1
- net IN3: track 85.2 -> 83.9 mm, vias 4 -> 2
- net SCK: track 23.7 -> 25.0 mm
- net MOSI: track 32.4 -> 33.6 mm
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